File: cc1101-2ch-dimmer.brd (EAGLE design)
At the start: 57.7 x 56.6 mm, 28 parts, among them Q1 IRLZ44NS, Q2 IRLZ44NS, U1 ATMEGA328P-AU, U2 0ZCG0035AF2C, U3 173950378, X2 MSTBA2, X3 MSTBA2, X4 MSTBA2, Y1 CSTCE8M00G52

Commit message: fixed wrong symbol for C3
Parts:
- C3: device rcl:R0805 -> rcl:C0805
Changed lines of the file:
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@@
 <element name="C1" library="rcl" library_urn="urn:adsk.eagle:library:334" package="C0805" package3d_urn="urn:adsk.eagle:package:23617/2" value="100n" x="23" y="40" smashed="yes" rot="R90">
 <attribute name="NAME" x="23" y="42.1254" size="1.27" layer="25" ratio="7" align="bottom-center"/>
+<attribute name="POPULARITY" value="88" x="23" y="40" size="1.778" layer="27" rot="R90" display="off"/>
 <attribute name="SPICEPREFIX" value="C" x="23" y="40" size="1.778" layer="27" rot="R90" display="off"/>
 <attribute name="VALUE" x="25.413" y="38.73" size="1.27" layer="27" rot="R90"/>
@@
 <element name="C2" library="rcl" library_urn="urn:adsk.eagle:library:334" package="C0805" package3d_urn="urn:adsk.eagle:package:23617/2" value="100n" x="18.2" y="23.3" smashed="yes" rot="R270">
 <attribute name="NAME" x="18.2" y="21.1746" size="1.27" layer="25" ratio="7" align="top-center"/>
+<attribute name="POPULARITY" value="88" x="18.2" y="23.3" size="1.778" layer="27" rot="R270" display="off"/>
 <attribute name="SPICEPREFIX" value="C" x="18.2" y="23.3" size="1.778" layer="27" rot="R270" display="off"/>
 <attribute name="VALUE" x="15.66" y="24.57" size="1.27" layer="27" rot="R270"/>
@@
 <attribute name="VALUE" x="15.48" y="56.375" size="1.27" layer="27" rot="R180"/>
 </element>
-<element name="C3" library="rcl" library_urn="urn:adsk.eagle:library:334" package="R0805" package3d_urn="urn:adsk.eagle:package:23553/2" value="100nF" x="30.8" y="34.3" smashed="yes" rot="R270">
+<element name="C3" library="rcl" library_urn="urn:adsk.eagle:library:334" package="C0805" package3d_urn="urn:adsk.eagle:package:23617/2" value="100nF" x="30.8" y="34.3" smashed="yes" rot="R270">
 <attribute name="NAME" x="31.8084" y="34.3" size="1.27" layer="25" ratio="7" align="center-left"/>
-<attribute name="SPICEPREFIX" value="R" x="25.8" y="34.3" size="1.778" layer="27" rot="R270" display="off"/>
+<attribute name="POPULARITY" value="88" x="30.8" y="34.3" size="1.778" layer="27" rot="R270" display="off"/>
+<attribute name="SPICEPREFIX" value="C" x="25.8" y="34.3" size="1.778" layer="27" rot="R270" display="off"/>
 <attribute name="VALUE" x="28.26" y="34.935" size="1.27" layer="27" rot="R270"/>
 </element>
@@
 <element name="C5" library="rcl" library_urn="urn:adsk.eagle:library:334" package="C0805" package3d_urn="urn:adsk.eagle:package:23617/2" value="100nF" x="30.8" y="41.1" smashed="yes" rot="R180">
 <attribute name="NAME" x="28.8016" y="41.1" size="1.27" layer="25" ratio="7" align="center-right"/>
+<attribute name="POPULARITY" value="88" x="30.8" y="41.1" size="1.778" layer="27" rot="R180" display="off"/>
 <attribute name="SPICEPREFIX" value="C" x="38.8" y="33.1" size="1.778" layer="27" rot="R180" display="off"/>
 <attribute name="VALUE" x="32.07" y="43.64" size="1.27" layer="27" rot="R180"/>
@@
 <element name="C4" library="rcl" library_urn="urn:adsk.eagle:library:334" package="C0805" package3d_urn="urn:adsk.eagle:package:23617/2" value="100n" x="10.7" y="40.9" smashed="yes">
 <attribute name="NAME" x="10.7" y="42.0354" size="1.27" layer="25" align="bottom-center"/>
+<attribute name="POPULARITY" value="88" x="10.7" y="40.9" size="1.778" layer="27" display="off"/>
 <attribute name="SPICEPREFIX" value="C" x="10.7" y="40.9" size="1.778" layer="27" display="off"/>
 <attribute name="VALUE" x="9.43" y="38.36" size="1.27" layer="27"/>
